File: hardware/BREAD_Slice.kicad_pcb (KiCad board)
At the start: 2 copper layers, 72.6 x 100 mm, 16 parts, among them J1 Conn_01x10_Female, J2 I2C_01x04

Commit message: Initial commit
Parts:
- added C10: 10 nF, Capacitor_SMD:C_1206_3216Metric_Pad1.33x1.80mm_HandSolder, B.Cu at (160.1, 119.8)
- added C11: 10 nF, Capacitor_SMD:C_1206_3216Metric_Pad1.33x1.80mm_HandSolder, B.Cu at (166.3, 114.0)
- added C12: 10 nF, Capacitor_SMD:C_1206_3216Metric_Pad1.33x1.80mm_HandSolder, B.Cu at (166.4, 74.1)
- added C5: 22uF, Capacitor_SMD:C_1206_3216Metric, B.Cu at (137.6, 60.8)
- added C6: 10 nF, Capacitor_SMD:C_1206_3216Metric_Pad1.33x1.80mm_HandSolder, B.Cu at (160.1, 61.6)
- added C7: 22uF, Capacitor_SMD:C_1206_3216Metric, B.Cu at (137.6, 57.8)
- added C8: 10 nF, Capacitor_SMD:C_1206_3216Metric_Pad1.33x1.80mm_HandSolder, B.Cu at (160.1, 79.8)
- added C9: 10 nF, Capacitor_SMD:C_1206_3216Metric_Pad1.33x1.80mm_HandSolder, B.Cu at (160.1, 101.5)
- added J10: Term_PressFit_Phoenix_Contact, SparkFun-Connector:Term_PressFit_5mm_H_PC, F.Cu at (180.6, 65.2)
- added J11: Term_PressFit_Phoenix_Contact, SparkFun-Connector:Term_PressFit_5mm_H_PC, F.Cu at (180.6, 70.2)
- added J12: cap, SparkFun-Connector:Term_PressFit_5mm_H_ENDCAP_PC, F.Cu at (180.6, 55.2)
- added J13: Term_PressFit_Phoenix_Contact, SparkFun-Connector:Term_PressFit_5mm_H_PC, F.Cu at (180.6, 60.2)
- added J14: cap, SparkFun-Connector:Term_PressFit_5mm_H_ENDCAP_PC, F.Cu at (180.6, 79.4)
- added J15: Term_PressFit_Phoenix_Contact, SparkFun-Connector:Term_PressFit_5mm_H_PC, F.Cu at (180.6, 84.4)
- added J16: Term_PressFit_Phoenix_Contact, SparkFun-Connector:Term_PressFit_5mm_H_PC, F.Cu at (180.6, 89.4)
- added J17: Term_PressFit_Phoenix_Contact, SparkFun-Connector:Term_PressFit_5mm_H_PC, F.Cu at (180.6, 94.4)
- added J18: I2C_01x04, Connector_JST:JST_SH_SM04B-SRSS-TB_1x04-1MP_P1.00mm_Horizontal, B.Cu at (142.6, 136.4)
- added J3: Term_PressFit_Phoenix_Contact, SparkFun-Connector:Term_PressFit_3.5mm_H_PC, F.Cu at (180.6, 120.6)
- added J4: Term_PressFit_Phoenix_Contact, SparkFun-Connector:Term_PressFit_3.5mm_H_PC, F.Cu at (180.6, 124.1)
- added J5: Term_PressFit_Phoenix_Contact, SparkFun-Connector:Term_PressFit_3.5mm_H_PC, F.Cu at (180.6, 127.6)
- added J6: cap, SparkFun-Connector:Term_PressFit_3.5mm_H_ENDCAP_PC, F.Cu at (180.6, 103.1)
- added J7: Term_PressFit_Phoenix_Contact, SparkFun-Connector:Term_PressFit_3.5mm_H_PC, F.Cu at (180.6, 106.6)
- added J8: Term_PressFit_Phoenix_Contact, SparkFun-Connector:Term_PressFit_3.5mm_H_PC, F.Cu at (180.6, 110.1)
- added J9: Term_PressFit_Phoenix_Contact, SparkFun-Connector:Term_PressFit_3.5mm_H_PC, F.Cu at (180.6, 113.6)
- added R1: 4.42 k, Resistor_SMD:R_1206_3216Metric_Pad1.30x1.75mm_HandSolder, B.Cu at (166.4, 76.8)
- added R2: 4.42 k, Resistor_SMD:R_1206_3216Metric_Pad1.30x1.75mm_HandSolder, B.Cu at (166.3, 116.7)
- added SW1: SW_SPDT, SparkFun-Switch:L102011MS02Q, F.Cu at (160.3, 55.6)
- added SW2: SW_SPDT, SparkFun-Switch:L102011MS02Q, F.Cu at (160.3, 95.9)
- added U2: AP63205WU-7, Package_TO_SOT_SMD:TSOT-23-6, B.Cu at (132.6, 64.2)
- added U3: LMD18200, Package_TO_SOT_THT:TO-220-11_P3.4x5.08mm_StaggerOdd_Lead4.85mm_Vertical, F.Cu at (156.6, 102.1)
- C2: value 100nF -> 10uF_t
- C3: value 22uF -> 10uF_t
- C4: value 22uF -> 100nF
- J2: value I2C_01x04 -> Term_PressFit_Phoenix_Contact; footprint Connector_JST:JST_SH_SM04B-SRSS-TB_1x04-1MP_P1.00mm_Horizontal -> SparkFun-Connector:Term_PressFit_3.5mm_H_PC; moved to F.Cu
- U1: value ~ -> LMD18200; footprint Package_TO_SOT_SMD:TSOT-23-6 -> Package_TO_SOT_THT:TO-220-11_P3.4x5.08mm_StaggerOdd_Lead4.85mm_Vertical; moved to F.Cu
- moved U1 66.6 mm to (156.6, 62.2), turned to -90 degrees
- moved C2 65.2 mm to (165.3, 70.7), turned to 0 degrees
- moved HS1 58.8 mm to (135.3, 62.7)
- moved C1 58.8 mm to (132.4, 60.8)
- moved L1 58.7 mm to (137.6, 64.2)
- moved C4 48.9 mm to (135.2, 67.6), turned to 180 degrees
- moved J2 36.0 mm to (180.6, 117.1), turned to 0 degrees
- moved C3 32.7 mm to (165.4, 110.6)
- moved A1 7.59 mm to (135.0, 100.0)
- moved Logo1 0.31 mm to (126.4, 72.4)
- renumbered D1 to D2, H3 to H2, H2 to H3
Connections:
- A1 pad 10: unconnected-(A1-D7-Pad10) -> /MC1
- A1 pad 11: unconnected-(A1-D8-Pad11) -> /BR1
- A1 pad 12: unconnected-(A1-D9-Pad12) -> /THRM1
- A1 pad 13: unconnected-(A1-D10-Pad13) -> /DIR2
- A1 pad 14: unconnected-(A1-D11-Pad14) -> /MC2
- A1 pad 15: unconnected-(A1-D12-Pad15) -> /BR2
- A1 pad 16: unconnected-(A1-D13-Pad16) -> /THRM2
- A1 pad 19: unconnected-(A1-A0-Pad19) -> /B2
- A1 pad 20: unconnected-(A1-A1-Pad20) -> /A2
- A1 pad 21: unconnected-(A1-A2-Pad21) -> /B1
- A1 pad 22: unconnected-(A1-A3-Pad22) -> /A1
- A1 pad 25: unconnected-(A1-A6-Pad25) -> /CSEN1
- A1 pad 26: unconnected-(A1-A7-Pad26) -> /CSEN2
- A1 pad 9: unconnected-(A1-D6-Pad9) -> /DIR1
- C2 pad 1: Net-(U1-SW) -> Net-(SW1-B)
- C2 pad 2: Net-(U1-BST) -> GND
- C3 pad 1: GND -> Net-(SW2-B)
- C3 pad 2: +5V -> GND
- C4 pad 1: GND -> Net-(U2-SW)
- C4 pad 2: +5V -> Net-(U2-BST)
- J2 pad 1: GND -> /A2
- L1 pad 1: Net-(U1-SW) -> Net-(U2-SW)
- U1 pad 1: +5V -> Net-(U1-BOOTSTRAP1)
- U1 pad 2: +12V -> Net-(U1-OUTPUT1)
- U1 pad 3: +12V -> /DIR1
- U1 pad 4: GND -> /BR1
- U1 pad 5: Net-(U1-SW) -> /MC1
- U1 pad 6: Net-(U1-BST) -> Net-(SW1-B)
Routing:
- net +12V: track 46.8 -> 129.3 mm
- net /BR1: track 0.00 -> 73.7 mm
- net /BR2: track 0.00 -> 72.8 mm
- net /THRM1: track 0.00 -> 67.1 mm
- net /MC1: track 0.00 -> 66.0 mm
- net /DIR1: track 0.00 -> 65.4 mm
- net +5V: track 108.9 -> 173.5 mm, vias 1 -> 2
- net /MC2: track 0.00 -> 64.3 mm
- net Net-(U3-OUTPUT2): track 0.00 -> 62.2 mm
- net /DIR2: track 0.00 -> 59.3 mm
- net /A1: track 0.00 -> 58.8 mm
- net /CUST2: track 0.00 -> 55.6 mm
- net /B1: track 0.00 -> 55.4 mm
- net /CSEN1: track 0.00 -> 52.1 mm, vias 0 -> 2
- net Net-(U1-OUTPUT2): track 0.00 -> 46.6 mm
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Other:
- board size 72.6 x 100 mm -> 70 x 100 mm
- board text added: "+"
- board text added: "-"
- board text added: "12V <-"
- board text added: "12V->5V Regulator"
- board text added: "5V"
- board text added: "A1"
- board text added: "A2"
- board text added: "B1"
- board text added: "B2"
- board text added: "BREAD Slice DC Motor Controller SLC_DCMT R1 2024"
- board text added: "CUSTOM PWR ->"
- board text added: "CUSTOM PWR 1"
- board text added: "CUSTOM PWR 2"
- board text added: "ENCODER 1"
- board text added: "ENCODER 2"
- board text added: "M1+"
- board text added: "M1-"
- board text added: "M2+"
- board text added: "M2-"
- board text added: "MOTOR 1"
- board text added: "MOTOR 2"
- board text added: "Motor 1"
- board text added: "Motor 2"
- board text removed: "12V->5V Reg"
- board text removed: "BREAD Slice Template SLC_TEMP <version> <year>"
