File: hardware/BREAD_Slice.kicad_pcb (KiCad board)
At the start: 2 copper layers, 70 x 100 mm, 38 parts, among them J1 Conn_01x10_Socket, J2 Screw_Terminal_01x04, J3 Screw_Terminal_01x04, J6 Screw_Terminal_01x02, J7 Screw_Terminal_01x02, J8 Screw_Terminal_01x02, J9 Screw_Terminal_01x02, U1 AP63205, U2 LMD18200T_NOPB, U3 LMD18200T_NOPB

Commit message: pcb almost finalized, needs switch and cap on lower driver shifted to route 12v rail
Parts:
- C11, C6, R1, R2: moved to F.Cu
- moved J7 59.7 mm to (188.6, 53.5)
- moved J6 59.5 mm to (188.6, 62.2)
- moved C10 58.7 mm to (176.3, 64.6)
- moved C12 58.7 mm to (180.5, 63.9)
- moved C13 58.7 mm to (157.4, 43.9)
- moved S2 58.7 mm to (161.3, 65.8)
- moved U3 58.7 mm to (155.2, 42.1)
- moved C14 58.7 mm to (156.9, 57.5)
- moved C5 58.3 mm to (176.7, 96.7)
- moved C7 58.3 mm to (180.8, 96.0)
- moved C8 58.3 mm to (157.8, 75.9)
- moved C9 58.3 mm to (157.2, 89.5)
- moved J4 58.3 mm to (188.6, 86.0)
- moved J5 58.3 mm to (188.6, 76.1)
- moved S1 58.3 mm to (161.7, 97.8)
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- renumbered J6 to J4, J8 to J5, J7 to J6, J9 to J7
Connections:
- A1 pad 10: /DIR1 -> /DIR2
- A1 pad 11: /BR1 -> /BR2
- A1 pad 12: /THRM1 -> /THRM2
- A1 pad 13: /PWM2 -> /PWM1
- A1 pad 14: /DIR2 -> /DIR1
- A1 pad 15: /BR2 -> /BR1
- A1 pad 16: /THRM2 -> /THRM1
- A1 pad 25: /CSENS1 -> /CSENS2
- A1 pad 26: /CSENS2 -> /CSENS1
- A1 pad 9: /PWM1 -> /PWM2
- J2 pad 1: /B1 -> /A1
- J2 pad 2: /A1 -> /B1
- J3 pad 1: /B2 -> /A2
- J3 pad 2: /A2 -> /B2
- J4 pad 2: +VDC -> /Motor Driver LMD185001/+VDC
- J6 pad 2: +VDC -> /Motor Driver LMD185002/+VDC
- S1 pad 3: +VDC -> /Motor Driver LMD185001/+VDC
- S2 pad 3: +VDC -> /Motor Driver LMD185002/+VDC
Routing:
- net /BR2: track 0.00 -> 88.9 mm
- net /DIR2: track 0.00 -> 82.9 mm
- net /PWM2: track 0.00 -> 80.6 mm, vias 0 -> 2
- net /THRM2: track 0.00 -> 74.8 mm
- net /BR1: track 0.00 -> 62.5 mm
- net /CSENS2: track 13.4 -> 73.5 mm, vias 1 -> 2
- net /DIR1: track 0.00 -> 58.3 mm, vias 0 -> 1
- net /PWM1: track 0.00 -> 56.4 mm
- net /THRM1: track 0.00 -> 47.8 mm, vias 0 -> 2
- net +5V: track 101.0 -> 142.5 mm
- net /B2: track 0.00 -> 34.9 mm
- net /A2: track 0.00 -> 34.9 mm
- net /B1: track 0.00 -> 32.2 mm
- net /A1: track 0.00 -> 32.2 mm
- net /CSENS1: track 13.4 -> 34.0 mm
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- added copper zone on F.Cu, net /Motor Driver LMD185001/+VDC
- added copper zone on F.Cu, net /Motor Driver LMD185002/+VDC
- removed copper zone on F.Cu, net +VDC
Other:
- board text added: "GND TIE"
