File: hardware/BREAD_Slice.kicad_sch (KiCad schematic)
At the start: 15 parts, among them J1 Conn_01x10_Female, J2 I2C_01x04

Commit message: Initial commit
Parts:
- removed J2: I2C_01x04, Connector_JST:JST_SH_SM04B-SRSS-TB_1x04-1MP_P1.00mm_Horizontal, symbol SparkFun-Connector:I2C_01x04
- removed U1: ~, Package_TO_SOT_SMD:TSOT-23-6, symbol SparkFun-DiscreteSemi:AP63205
- added C10, C11, C12, C6, C8, C9: 10 nF, Capacitor_SMD:C_1206_3216Metric_Pad1.33x1.80mm_HandSolder, symbol Device:C
- added C2, C3: 10uF_t, Capacitor_SMD:C_1206_3216Metric, symbol BREAD_Slice-rescue:10uF_t-OCI_UPL_2_Capacitors
- added J10, J11, J13, J15, J16, J17: Term_PressFit_Phoenix_Contact, SparkFun-Connector:Term_PressFit_5mm_H_PC, symbol SparkFun-Connector:Term_PressFit_Phoenix_Contact
- added J12, J14: Term_PressFit_Phoenix_Contact, SparkFun-Connector:Term_PressFit_5mm_H_ENDCAP_PC, symbol SparkFun-Connector:Term_PressFit_Phoenix_Contact
- added J18: I2C_01x04, Connector_JST:JST_SH_SM04B-SRSS-TB_1x04-1MP_P1.00mm_Horizontal, symbol SparkFun-Connector:I2C_01x04
- added J2, J3, J4, J5, J7, J8, J9: Term_PressFit_Phoenix_Contact, SparkFun-Connector:Term_PressFit_3.5mm_H_PC, symbol SparkFun-Connector:Term_PressFit_Phoenix_Contact
- added J6: Term_PressFit_Phoenix_Contact, SparkFun-Connector:Term_PressFit_3.5mm_H_ENDCAP_PC, symbol SparkFun-Connector:Term_PressFit_Phoenix_Contact
- added Logo1: Logo_Open_Hardware_Small, Symbol:OSHW-Symbol_6.7x6mm_SilkScreen, symbol Graphic:Logo_Open_Hardware_Small
- added R1, R2: 4.42 k, Resistor_SMD:R_1206_3216Metric_Pad1.30x1.75mm_HandSolder, symbol Device:R
- added SW1, SW2: SW_SPDT, SparkFun-Switch:L102011MS02Q, symbol Switch:SW_SPDT
- added U1, U3: LMD18200, Package_TO_SOT_THT:TO-220-11_P3.4x5.08mm_StaggerOdd_Lead4.85mm_Vertical, symbol Driver_Motor:LMD18200
- added U2: AP63205WU-7, Package_TO_SOT_SMD:TSOT-23-6, symbol SparkFun-DiscreteSemi:AP63205
- renumbered C2 to C4, C3 to C5, C4 to C7, D1 to D2, H3 to H2, H2 to H3
Connections:
- net +12V: now also SW1.1 (A), SW2.1 (A), U2.2 (EN), U2.3 (VIN)
- net +5V: now also J18.2 (Pin_2), J4.1, J8.1, U2.1 (FB)
- net GND: now also C11.2, C12.2, C2.2, C3.2, J11.1, J17.1, J18.1 (Pin_1), J5.1, J9.1, R1.2, R2.2, U1.7 (GND), U2.4 (GND), U3.7 (GND)
- net I2C_CLK: now also J18.4 (Pin_4)
- net I2C_DAT: now also J18.3 (Pin_3)
- net MC1: now reaches A1.10 (D7)
- net MC1: now also U1.5 (PWM)
- net BR1: now reaches A1.11 (D8)
- net BR1: now also U1.4 (BRAKE)
- net THRM1: now reaches A1.12 (D9)
- net THRM1: now also U1.9 (~{THERMAL_FLAG_OUTPUT})
- net DIR2: now reaches A1.13 (D10)
- net DIR2: now also U3.3 (DIRECTION)
- net MC2: now reaches A1.14 (D11)
- net MC2: now also U3.5 (PWM)
- net BR2: now reaches A1.15 (D12)
- net BR2: now also U3.4 (BRAKE)
- net THRM2: now reaches A1.16 (D13)
- net THRM2: now also U3.9 (~{THERMAL_FLAG_OUTPUT})
- net B2: now reaches A1.19 (A0)
- net B2: now also J3.1
- net A2: now reaches A1.20 (A1)
- net A2: now also J2.1
- net B1: now reaches A1.21 (A2)
- net B1: now also J7.1
- net A1: now reaches A1.22 (A3)
- net A1: now also J6.1
- net CSEN1: now reaches A1.25 (A6)
- net CSEN1: now also C12.1, R1.1, U1.8 (CURRENT_SENSE_OUTPUT)
- net CSEN2: now reaches A1.26 (A7)
- net CSEN2: now also C11.1, R2.1, U3.8 (CURRENT_SENSE_OUTPUT)
- net DIR1: now reaches A1.9 (D6)
- net DIR1: now also U1.3 (DIRECTION)
- net at C4.1, L1.1: now also U2.5 (SW)
- net at C4.2: now also U2.6 (BST)
- new net: C10.1, U3.11 (BOOTSTRAP2)
- new net: C10.2, J15.1, U3.10 (OUTPUT2)
- new net: C8.1, U1.11 (BOOTSTRAP2)
- new net: C8.2, J13.1, U1.10 (OUTPUT2)
- new net: C9.1, J14.1, U3.2 (OUTPUT1)
- new net: C9.2, U3.1 (BOOTSTRAP1)
- new net: C3.1, SW2.2 (B), U3.6 (VS)
- new net: C2.1, SW1.2 (B), U1.6 (VS)
- new net: C6.2, U1.1 (BOOTSTRAP1)
- new net: C6.1, J12.1, U1.2 (OUTPUT1)
- new net CUST1: J10.1, SW1.3 (C)
- new net CUST2: J16.1, SW2.3 (C)
- no-connect marks 22 -> 7
Other:
- note added: "Current sensing resistor R = 5V / (377uA/A*3A) = 4.42k"
- moved on the sheet: A1, C1, C4, C5, C7, D2, H1, H2, H3, H4, J1, L1
