File: hardware/BREAD_Slice.kicad_sch (KiCad schematic)
At the start: 17 parts, among them J1 Conn_01x10_Socket, J2 Screw_Terminal_01x04, J3 Screw_Terminal_01x04, U1 AP63205

Commit message: pcb almost finalized, needs switch and cap on lower driver shifted to route 12v rail
Connections:
- net A1: now also J2.1 (Pin_1); no longer J2.2 (Pin_2)
- net A2: now also J3.1 (Pin_1); no longer J3.2 (Pin_2)
- net B1: now also J2.2 (Pin_2); no longer J2.1 (Pin_1)
- net B2: now also J3.2 (Pin_2); no longer J3.1 (Pin_1)
- net BR1: now also A1.15 (D12); no longer A1.11 (D8)
- net BR2: now also A1.11 (D8); no longer A1.15 (D12)
- net CSENS1: now also A1.26 (A7); no longer A1.25 (A6)
- net CSENS2: now also A1.25 (A6); no longer A1.26 (A7)
- net DIR1: now also A1.14 (D11); no longer A1.10 (D7)
- net DIR2: now also A1.10 (D7); no longer A1.14 (D11)
- net PWM1: now also A1.13 (D10); no longer A1.9 (D6)
- net PWM2: now also A1.9 (D6); no longer A1.13 (D10)
- net THRM1: now also A1.16 (D13); no longer A1.12 (D9)
- net THRM2: now also A1.12 (D9); no longer A1.16 (D13)

Commit message: review and revise for current template and kmlib
Parts:
- D1: footprint SparkFun-LED:WS2812-5050-4PIN -> KMLib_IC_SMD:WS2812-5050-4PIN
- HS1: footprint kml-custom:Thermal Pad -> KMLib_Mounting:Thermal Pad
- U1: footprint kml-custom:SOIC_05WU-7_DIO -> KMLib_IC_SMD:SOIC_05WU-7_DIO; symbol kml-custom:AP63205WU-7 -> KMLib_IC_Power:AP63205WU-7_Buck_Regulator
Changed lines of the file:
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@@
 			)
 		)
-		(property "Description" ""
+		(property "Description" "Mounting Hole without connection"
 			(at 49.53 185.42 0)
 			(effects
@@
 			)
 		)
-		(property "Description" ""
+		(property "Description" "Mounting Hole without connection"
 			(at 49.53 190.5 0)
 			(effects
@@
 			)
 		)
-		(property "Description" ""
+		(property "Description" "Mounting Hole without connection"
 			(at 57.15 185.42 0)
 			(effects
@@
 			)
 		)
-		(property "Description" ""
+		(property "Description" "Mounting Hole without connection"
 			(at 57.15 190.5 0)
 			(effects
@@
 			)
 		)
-		(property "Description" ""
+		(property "Description" "Arduino Nano v3.x"
 			(at 40.64 143.51 0)
 			(effects
@@
 			)
 		)
-		(property "Description" ""
+		(property "Description" "Unpolarized capacitor, small symbol"
 			(at 52.07 72.39 0)
 			(effects
@@
 			)
 		)
-		(property "Description" ""
+		(property "Description" "Unpolarized capacitor, small symbol"
 			(at 52.07 82.55 0)
 			(effects
@@
 	)
 	(symbol
-		(lib_id "kml-custom:AP63205WU-7")
+		(lib_id "KMLib_IC_Power:AP63205WU-7_Buck_Regulator")
 		(at 35.56 73.66 0)
 		(unit 1)
@@
 			)
 		)
-		(property "Footprint" "kml-custom:SOIC_05WU-7_DIO"
+		(property "Footprint" "KMLib_IC_SMD:SOIC_05WU-7_DIO"
 			(at 35.56 73.66 0)
 			(effects
@@
 	)
 	(symbol
-		(lib_name "WS2812B_5050_1")
 		(lib_id "SparkFun-LED:WS2812B_5050")
 		(at 30.48 40.64 0)
@@
 			)
 		)
-		(property "Footprint" "SparkFun-LED:WS2812-5050-4PIN"
+		(property "Footprint" "KMLib_IC_SMD:WS2812-5050-4PIN"
 			(at 13.97 49.53 0)
 			(effects
@@
 	)
 	(symbol
-		(lib_name "+12V_2")
 		(lib_id "power:+12V")
 		(at 86.36 114.3 0)
@@
 	)
 	(symbol
-		(lib_name "+12V_1")
 		(lib_id "power:+12V")
 		(at 53.34 27.94 0)
@@
 	)
 	(symbol
-		(lib_name "+12V_2")
 		(lib_id "power:+12V")
 		(at 26.67 69.85 0)
@@
 			)
 		)
-		(property "Footprint" "kml-custom:Thermal Pad"
+		(property "Footprint" "KMLib_Mounting:Thermal Pad"
 			(at 35.8648 97.79 0)
 			(effects
@@
 			)
 		)
-		(property "Description" ""
+		(property "Description" "Inductor, small symbol"
 			(at 52.07 77.47 0)
 			(effects
@@
 	)
 	(symbol
-		(lib_name "+12V_2")
 		(lib_id "power:+12V")
 		(at 86.36 39.37 0)
@@
 			)
 		)
-		(property "Description" ""
+		(property "Description" "Unpolarized capacitor, small symbol"
 			(at 62.23 82.55 0)
 			(effects
@@
 			)
 		)
-		(property "Description" ""
+		(property "Description" "Unpolarized capacitor, small symbol"
 			(at 26.67 80.01 0)
 			(effects
