File: hardware/BREAD_Slice.kicad_sch (KiCad schematic)
At the start: 17 parts, among them J1 Conn_01x10_Socket, J2 Screw_Terminal_01x04, J3 Screw_Terminal_01x04, U1 AP63205

Commit message: feat: update to kicad 10 and migrate old references to kml
Parts:
- D1: symbol SparkFun-LED:WS2812B_5050 -> KMLib_IC_Digital:WS2812B_5050_RGB_LED
- HS1: footprint KMLib_Mounting:Thermal Pad -> KMLib_Mounting:Thermal_Pad
