File: archive/hw_archive/2021-06-08/BREAD_Slice.kicad_pcb (KiCad board)
At the start: 2 copper layers, 70 x 100 mm, 30 parts, among them J1 Conn_01x10_Female, J2 Screw_Terminal_01x04, J3 Screw_Terminal_01x04, J4 Conn_01x03_Male, J5 Conn_01x03_Male, J6 Screw_Terminal_01x02, J7 Screw_Terminal_01x02, J8 Screw_Terminal_01x02, J9 Screw_Terminal_01x02, U1 LMD18200, U2 LMD18200

Commit message: chore(archive): upgrade the archived board files to the KiCad 10 format
The archived projects were last saved by KiCad 5.1 (2021-06-08), 6.x
(2023-12-13) and 9.0 (recent_finn), and no longer load cleanly in the
current toolchain. All three are now saved by KiCad 10.0.6, so they can
be opened, netlisted and DRC-checked without a per-file conversion step.

The upgrade changes format only. Verified per board by normalizing both
revisions out of the s-expressions and diffing:

- pad -> net map identical (112, 112, 134 pads)
- track, arc and via geometry identical (198, 198, 322 items)
- net name sets identical apart from the unnamed net 0, which KiCad 10
  no longer emits on pad references

No copper, footprint or connectivity was edited.

The 2021-06-08 project also gains .kicad_sch, .kicad_pro and .kicad_prl,
converted by KiCad from the legacy .sch and .pro. The legacy .sch, .pro,
.net and -cache.lib files are retained alongside them as the
as-fabricated record.
Other:
- net class Default removed
