File: archive/hw_archive/2021-06-08/BREAD_Slice.kicad_sch (KiCad schematic)
At the start: 29 parts, among them J1 Conn_01x10_Female, J2 Screw_Terminal_01x04, J3 Screw_Terminal_01x04, J4 Conn_01x03_Pin, J5 Conn_01x03_Pin, J6 Screw_Terminal_01x02, J7 Screw_Terminal_01x02, J8 Screw_Terminal_01x02, J9 Screw_Terminal_01x02, U1 LMD18200, U2 LMD18200

Commit message: chore(archive): upgrade the archived board files to the KiCad 10 format
The archived projects were last saved by KiCad 5.1 (2021-06-08), 6.x
(2023-12-13) and 9.0 (recent_finn), and no longer load cleanly in the
current toolchain. All three are now saved by KiCad 10.0.6, so they can
be opened, netlisted and DRC-checked without a per-file conversion step.

The upgrade changes format only. Verified per board by normalizing both
revisions out of the s-expressions and diffing:

- pad -> net map identical (112, 112, 134 pads)
- track, arc and via geometry identical (198, 198, 322 items)
- net name sets identical apart from the unnamed net 0, which KiCad 10
  no longer emits on pad references

No copper, footprint or connectivity was edited.

The 2021-06-08 project also gains .kicad_sch, .kicad_pro and .kicad_prl,
converted by KiCad from the legacy .sch and .pro. The legacy .sch, .pro,
.net and -cache.lib files are retained alongside them as the
as-fabricated record.
Parts:
- removed C3, C4: 10uF_t, symbol Device:C
- removed J4, J5: Conn_01x03_Pin, symbol Connector:Conn_01x03_Pin
- added C3, C4: 10uF_t, OCI_UPL_FOOTPRINTS:C_2312, symbol OCI_UPL_2_Capacitors:10uF_t
- added J4, J5: Conn_01x03_Male, Connector_PinSocket_2.54mm:PinSocket_1x03_P2.54mm_Vertical, symbol Connector:Conn_01x03_Male
- C1, C2: symbol BREAD_Slice-rescue:10uF_t-OCI_UPL_2_Capacitors -> OCI_UPL_2_Capacitors:10uF_t
- J1: symbol BREAD_Slice-rescue:Conn_01x10_Female-Connector -> Connector:Conn_01x10_Female
Connections:
- net +12V: now also C1.1, J1.2 (Pin_2), J1.9 (Pin_9), J4.2 (Pin_2), J5.2 (Pin_2)
- net +5V: now also C2.1
- net CUST1: now also J4.1 (Pin_1)
- net CUST2: now also J5.1 (Pin_1)
- net E_STOP: now also J1.6 (Pin_6)
- net GND: now also C1.2, C2.2, J1.1 (Pin_1), J1.10 (Pin_10), J1.5 (Pin_5), C3.2, C4.2
- net I2C_CLK: now also J1.3 (Pin_3)
- net I2C_DAT: now also J1.4 (Pin_4)
- net INT: now also J1.7 (Pin_7)
- net SYNC: now also J1.8 (Pin_8)
- net at U1.6 (VS): now also C3.1, J4.3 (Pin_3)
- net at U2.6 (VS): now also C4.1, J5.3 (Pin_3)
Other:
- moved on the sheet: C10, C5, C6, C7, C8, C9, J6, J7, J8, J9, R3, R4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
